File: MiniCurso.sch (KiCad schematic (older format))
At the start: 4 parts

Commit message: add crystal, UCAP and bypass caps
Parts:
- added C? (x2): 15p, symbol Device:C
- added C? (x2): 1u, symbol Device:C
- added C? (x2): 100n, symbol Device:C
- added Y?: 16MHz, symbol Device:Crystal
Connections:
- wire segments 7 -> 19

Commit message: add reset, pin headers
Parts:
- added C?: 100n, symbol Device:C
- added J? (x2): Conn_01x10, symbol Connector_Generic:Conn_01x10
- added J?: Conn_01x06, symbol Connector_Generic:Conn_01x06
- added R?: 10k, symbol Device:R
- added SW?: SW_Push, symbol Switch:SW_Push
Connections:
- wire segments 19 -> 52
Changed lines of the file:
@@
 	1    0    0    -1
 $EndComp
+$Comp
+L Switch:SW_Push SW?
+U 1 1 5D7A722F
+P 3850 2450
+F 0 "SW?" H 3850 2735 50  0000 C CNN
+F 1 "SW_Push" H 3850 2644 50  0000 C CNN
+F 2 "" H 3850 2650 50  0001 C CNN
+F 3 "" H 3850 2650 50  0001 C CNN
+	1    3850 2450
+	1    0    0    -1
+$EndComp
+Wire Wire Line
+	4050 2450 4150 2450
+$Comp
+L power:GND #PWR?
+U 1 1 5D7A7443
+P 3650 2450
+F 0 "#PWR?" H 3650 2200 50  0001 C CNN
+F 1 "GND" V 3655 2322 50  0000 R CNN
+F 2 "" H 3650 2450 50  0001 C CNN
+F 3 "" H 3650 2450 50  0001 C CNN
+	1    3650 2450
+	0    1    1    0
+$EndComp
+$Comp
+L power:+5V #PWR?
+U 1 1 5D7A747E
+P 4150 2150
+F 0 "#PWR?" H 4150 2000 50  0001 C CNN
+F 1 "+5V" H 4165 2323 50  0000 C CNN
+F 2 "" H 4150 2150 50  0001 C CNN
+F 3 "" H 4150 2150 50  0001 C CNN
+	1    4150 2150
+	1    0    0    -1
+$EndComp
+$Comp
+L Device:R R?
+U 1 1 5D7A74A1
+P 4150 2300
+F 0 "R?" V 3950 2300 50  0000 C CNN
+F 1 "10k" V 4050 2300 50  0000 C CNN
+F 2 "" V 4080 2300 50  0001 C CNN
+F 3 "~" H 4150 2300 50  0001 C CNN
+	1    4150 2300
+	-1   0    0    1
+$EndComp
+$Comp
+L Device:C C?
+U 1 1 5D7A7D7B
+P 4150 2600
+F 0 "C?" H 4265 2646 50  0000 L CNN
+F 1 "100n" H 4265 2555 50  0000 L CNN
+F 2 "" H 4188 2450 50  0001 C CNN
+F 3 "~" H 4150 2600 50  0001 C CNN
+	1    4150 2600
+	1    0    0    -1
+$EndComp
+Connection ~ 4150 2450
+$Comp
+L power:GND #PWR?
+U 1 1 5D7A7DD1
+P 4150 2750
+F 0 "#PWR?" H 4150 2500 50  0001 C CNN
+F 1 "GND" H 4155 2577 50  0000 C CNN
+F 2 "" H 4150 2750 50  0001 C CNN
+F 3 "" H 4150 2750 50  0001 C CNN
+	1    4150 2750
+	1    0    0    -1
+$EndComp
+Wire Wire Line
+	4150 2450 5200 2450
+Wire Wire Line
+	5200 2450 5200 2900
+$Comp
+L Connector_Generic:Conn_01x10 J?
+U 1 1 5D7A93D5
+P 6900 3300
+F 0 "J?" H 6980 3292 50  0000 L CNN
+F 1 "Conn_01x10" H 6980 3201 50  0000 L CNN
+F 2 "" H 6900 3300 50  0001 C CNN
+F 3 "~" H 6900 3300 50  0001 C CNN
+	1    6900 3300
+	1    0    0    -1
+$EndComp
+$Comp
+L Connector_Generic:Conn_01x10 J?
+U 1 1 5D7A94CD
+P 6900 4500
+F 0 "J?" H 6980 4492 50  0000 L CNN
+F 1 "Conn_01x10" H 6980 4401 50  0000 L CNN
+F 2 "" H 6900 4500 50  0001 C CNN
+F 3 "~" H 6900 4500 50  0001 C CNN
+	1    6900 4500
+	1    0    0    -1
+$EndComp
+$Comp
+L Connector_Generic:Conn_01x06 J?
+U 1 1 5D7A9629
+P 6900 5500
+F 0 "J?" H 6980 5492 50  0000 L CNN
+F 1 "Conn_01x06" H 6980 5401 50  0000 L CNN
+F 2 "" H 6900 5500 50  0001 C CNN
+F 3 "~" H 6900 5500 50  0001 C CNN
+	1    6900 5500
+	1    0    0    -1
+$EndComp
+Wire Wire Line
+	6700 5800 6400 5800
+Wire Wire Line
+	6700 5700 6400 5700
+Wire Wire Line
+	6700 5600 6400 5600
+Wire Wire Line
+	6700 5500 6400 5500
+Wire Wire Line
+	6700 5400 6400 5400
+Wire Wire Line
+	6700 5300 6400 5300
+Wire Wire Line
+	6400 4100 6700 4100
+Wire Wire Line
+	6400 4200 6700 4200
+Wire Wire Line
+	6400 4300 6700 4300
+Wire Wire Line
+	6400 4400 6700 4400
+Wire Wire Line
+	6400 4500 6700 4500
+Wire Wire Line
+	6400 4600 6700 4600
+Wire Wire Line
+	6400 4700 6700 4700
+Wire Wire Line
+	6400 4800 6700 4800
+Wire Wire Line
+	6400 5000 6400 4900
+Wire Wire Line
+	6400 4900 6700 4900
+Wire Wire Line
+	6400 5100 6700 5100
+Wire Wire Line
+	6700 5100 6700 5000
+Wire Wire Line
+	6400 3900 6700 3900
+Wire Wire Line
+	6700 3900 6700 3800
+Wire Wire Line
+	6400 3800 6400 3700
+Wire Wire Line
+	6400 3700 6700 3700
+Wire Wire Line
+	6400 3600 6700 3600
+Wire Wire Line
+	6400 3500 6700 3500
+Wire Wire Line
+	6400 3400 6700 3400
+Wire Wire Line
+	6400 3300 6700 3300
+Wire Wire Line
+	6400 3200 6700 3200
+Wire Wire Line
+	6400 3100 6700 3100
+Wire Wire Line
+	6400 3000 6700 3000
+Wire Wire Line
+	6400 2900 6700 2900
 $EndSCHEMATC

Commit message: annotated components
	-the components were added by KiCads automatic annotate feature.
Parts:
- gave numbers to parts that had none: 17
Changed lines of the file:
@@
 $EndDescr
 $Comp
-L MCU_Microchip_ATmega:ATmega32U4-AU U?
+L MCU_Microchip_ATmega:ATmega32U4-AU U1
 U 1 1 5D7A3850
 P 5800 4400
-F 0 "U?" H 5800 2200 50  0000 C CNN
+F 0 "U1" H 5800 2200 50  0000 C CNN
 F 1 "ATmega32U4-AU" H 5800 2100 50  0000 C CNN
 F 2 "Package_QFP:TQFP-44_10x10mm_P0.8mm" H 5800 4400 50  0001 C CIN
@@
 $EndComp
 $Comp
-L power:+5V #PWR?
+L power:+5V #PWR05
 U 1 1 5D7A41BE
 P 4250 3500
-F 0 "#PWR?" H 4250 3350 50  0001 C CNN
+F 0 "#PWR05" H 4250 3350 50  0001 C CNN
 F 1 "+5V" H 4265 3673 50  0000 C CNN
 F 2 "" H 4250 3500 50  0001 C CNN
@@
 $EndComp
 $Comp
-L Connector:USB_B_Micro J?
+L Connector:USB_B_Micro J1
 U 1 1 5D7A43C6
 P 3750 3900
-F 0 "J?" H 3750 4450 50  0000 C CNN
+F 0 "J1" H 3750 4450 50  0000 C CNN
 F 1 "USB_B_Micro" H 3750 4300 50  0000 C CNN
 F 2 "" H 3900 3850 50  0001 C CNN
@@
 	4250 3700 4050 3700
 $Comp
-L Device:R R?
+L Device:R R2
 U 1 1 5D7A444B
 P 4600 3900
-F 0 "R?" V 4400 3900 50  0000 C CNN
+F 0 "R2" V 4400 3900 50  0000 C CNN
 F 1 "22R" V 4500 3900 50  0000 C CNN
 F 2 "" V 4530 3900 50  0001 C CNN
@@
 $EndComp
 $Comp
-L Device:R R?
+L Device:R R3
 U 1 1 5D7A44FE
 P 4600 4000
-F 0 "R?" V 4800 4000 50  0000 C CNN
+F 0 "R3" V 4800 4000 50  0000 C CNN
 F 1 "22R" V 4700 4000 50  0000 C CNN
 F 2 "" V 4530 4000 50  0001 C CNN
@@
 	4450 3900 4050 3900
 $Comp
-L power:GND #PWR?
+L power:GND #PWR02
 U 1 1 5D7A4BCB
 P 3750 4550
-F 0 "#PWR?" H 3750 4300 50  0001 C CNN
+F 0 "#PWR02" H 3750 4300 50  0001 C CNN
 F 1 "GND" H 3755 4377 50  0000 C CNN
 F 2 "" H 3750 4550 50  0001 C CNN
@@
 	3750 4550 3750 4300
 $Comp
-L power:+5V #PWR?
+L power:+5V #PWR010
 U 1 1 5D7A4D0F
 P 5800 2200
-F 0 "#PWR?" H 5800 2050 50  0001 C CNN
+F 0 "#PWR010" H 5800 2050 50  0001 C CNN
 F 1 "+5V" H 5815 2373 50  0000 C CNN
 F 2 "" H 5800 2200 50  0001 C CNN
@@
 	5700 2200 5700 2600
 $Comp
-L power:GND #PWR?
+L power:GND #PWR011
 U 1 1 5D7A5158
 P 5800 6300
-F 0 "#PWR?" H 5800 6050 50  0001 C CNN
+F 0 "#PWR011" H 5800 6050 50  0001 C CNN
 F 1 "GND" H 5805 6127 50  0000 C CNN
 F 2 "" H 5800 6300 50  0001 C CNN
@@
 Connection ~ 5800 6300
 $Comp
-L Device:Crystal Y?
+L Device:Crystal Y1
 U 1 1 5D7A5555
 P 4900 3200
-F 0 "Y?" V 4950 3500 50  0000 R CNN
+F 0 "Y1" V 4950 3500 50  0000 R CNN
 F 1 "16MHz" V 4850 3600 50  0000 R CNN
 F 2 "" H 4900 3200 50  0001 C CNN
@@
 	5200 3350 5200 3300
 $Comp
-L Device:C C?
+L Device:C C2
 U 1 1 5D7A5966
 P 4900 2900
-F 0 "C?" H 5015 2946 50  0000 L CNN
+F 0 "C2" H 5015 2946 50  0000 L CNN
 F 1 "15p" H 5015 2855 50  0000 L CNN
 F 2 "" H 4938 2750 50  0001 C CNN
@@
 Connection ~ 4900 3050
 $Comp
-L Device:C C?
+L Device:C C3
 U 1 1 5D7A599C
 P 4900 3500
-F 0 "C?" H 5015 3546 50  0000 L CNN
+F 0 "C3" H 5015 3546 50  0000 L CNN
 F 1 "15p" H 5015 3455 50  0000 L CNN
 F 2 "" H 4938 3350 50  0001 C CNN
@@
 Connection ~ 4900 3350
 $Comp
-L power:GND #PWR?
+L power:GND #PWR07
 U 1 1 5D7A5BF0
 P 4900 3650
-F 0 "#PWR?" H 4900 3400 50  0001 C CNN
+F 0 "#PWR07" H 4900 3400 50  0001 C CNN
 F 1 "GND" H 4905 3477 50  0000 C CNN
 F 2 "" H 4900 3650 50  0001 C CNN
@@
 $EndComp
 $Comp
-L power:GND #PWR?
+L power:GND #PWR06
 U 1 1 5D7A5C10
 P 4900 2750
-F 0 "#PWR?" H 4900 2500 50  0001 C CNN
+F 0 "#PWR06" H 4900 2500 50  0001 C CNN
 F 1 "GND" H 4905 2577 50  0000 C CNN
 F 2 "" H 4900 2750 50  0001 C CNN
@@
 $EndComp
 $Comp
-L power:+5V #PWR?
+L power:+5V #PWR09
 U 1 1 5D7A6172
 P 5200 3700
-F 0 "#PWR?" H 5200 3550 50  0001 C CNN
+F 0 "#PWR09" H 5200 3550 50  0001 C CNN
 F 1 "+5V" V 5100 3700 50  0000 L CNN
 F 2 "" H 5200 3700 50  0001 C CNN
@@
 $EndComp
 $Comp
-L Device:C C?
+L Device:C C4
 U 1 1 5D7A633C
 P 5050 4200
-F 0 "C?" V 5200 4200 50  0000 C CNN
+F 0 "C4" V 5200 4200 50  0000 C CNN
 F 1 "1u" V 5300 4200 50  0000 C CNN
 F 2 "" H 5088 4050 50  0001 C CNN
@@
 $EndComp
 $Comp
-L power:GND #PWR?
+L power:GND #PWR08
 U 1 1 5D7A64DF
 P 4900 4200
-F 0 "#PWR?" H 4900 3950 50  0001 C CNN
+F 0 "#PWR08" H 4900 3950 50  0001 C CNN
 F 1 "GND" V 5000 4200 50  0000 R CNN
 F 2 "" H 4900 4200 50  0001 C CNN
@@
 $EndComp
 $Comp
-L Device:C C?
+L Device:C C5
 U 1 1 5D7A6CDC
 P 6250 2100
-F 0 "C?" H 6365 2146 50  0000 L CNN
+F 0 "C5" H 6365 2146 50  0000 L CNN
 F 1 "1u" H 6365 2055 50  0000 L CNN
 F 2 "" H 6288 1950 50  0001 C CNN
@@
 $EndComp
 $Comp
-L Device:C C?
+L Device:C C6
 U 1 1 5D7A6D34
 P 6650 2100
-F 0 "C?" H 6765 2146 50  0000 L CNN
+F 0 "C6" H 6765 2146 50  0000 L CNN
 F 1 "100n" H 6765 2055 50  0000 L CNN
 F 2 "" H 6688 1950 50  0001 C CNN
@@
 $EndComp
 $Comp
-L Device:C C?
+L Device:C C7
 U 1 1 5D7A6D64
 P 7050 2100
-F 0 "C?" H 7165 2146 50  0000 L CNN
+F 0 "C7" H 7165 2146 50  0000 L CNN
 F 1 "100n" H 7165 2055 50  0000 L CNN
 F 2 "" H 7088 1950 50  0001 C CNN
@@
 $EndComp
 $Comp
-L power:+5V #PWR?
+L power:+5V #PWR012
 U 1 1 5D7A6DA2
 P 6250 1950
-F 0 "#PWR?" H 6250 1800 50  0001 C CNN
+F 0 "#PWR012" H 6250 1800 50  0001 C CNN
 F 1 "+5V" H 6265 2123 50  0000 C CNN
 F 2 "" H 6250 1950 50  0001 C CNN
@@
 $EndComp
 $Comp
-L power:+5V #PWR?
+L power:+5V #PWR014
 U 1 1 5D7A6DC3
 P 6650 1950
-F 0 "#PWR?" H 6650 1800 50  0001 C CNN
+F 0 "#PWR014" H 6650 1800 50  0001 C CNN
 F 1 "+5V" H 6665 2123 50  0000 C CNN
 F 2 "" H 6650 1950 50  0001 C CNN
@@
 $EndComp
 $Comp
-L power:+5V #PWR?
+L power:+5V #PWR016
 U 1 1 5D7A6DE4
 P 7050 1950
-F 0 "#PWR?" H 7050 1800 50  0001 C CNN
+F 0 "#PWR016" H 7050 1800 50  0001 C CNN
 F 1 "+5V" H 7065 2123 50  0000 C CNN
 F 2 "" H 7050 1950 50  0001 C CNN
@@
 $EndComp
 $Comp
-L power:GND #PWR?
+L power:GND #PWR013
 U 1 1 5D7A6E05
 P 6250 2250
-F 0 "#PWR?" H 6250 2000 50  0001 C CNN
+F 0 "#PWR013" H 6250 2000 50  0001 C CNN
 F 1 "GND" H 6255 2077 50  0000 C CNN
 F 2 "" H 6250 2250 50  0001 C CNN
@@
 $EndComp
 $Comp
-L power:GND #PWR?
+L power:GND #PWR015
 U 1 1 5D7A6E3C
 P 6650 2250
-F 0 "#PWR?" H 6650 2000 50  0001 C CNN
+F 0 "#PWR015" H 6650 2000 50  0001 C CNN
 F 1 "GND" H 6655 2077 50  0000 C CNN
 F 2 "" H 6650 2250 50  0001 C CNN
@@
 $EndComp
 $Comp
-L power:GND #PWR?
+L power:GND #PWR017
 U 1 1 5D7A6E5D
 P 7050 2250
-F 0 "#PWR?" H 7050 2000 50  0001 C CNN
+F 0 "#PWR017" H 7050 2000 50  0001 C CNN
 F 1 "GND" H 7055 2077 50  0000 C CNN
 F 2 "" H 7050 2250 50  0001 C CNN
@@
 $EndComp
 $Comp
-L Switch:SW_Push SW?
+L Switch:SW_Push SW1
 U 1 1 5D7A722F
 P 3850 2450
-F 0 "SW?" H 3850 2735 50  0000 C CNN
+F 0 "SW1" H 3850 2735 50  0000 C CNN
 F 1 "SW_Push" H 3850 2644 50  0000 C CNN
 F 2 "" H 3850 2650 50  0001 C CNN
@@
 	4050 2450 4150 2450
 $Comp
-L power:GND #PWR?
+L power:GND #PWR01
 U 1 1 5D7A7443
 P 3650 2450
-F 0 "#PWR?" H 3650 2200 50  0001 C CNN
+F 0 "#PWR01" H 3650 2200 50  0001 C CNN
 F 1 "GND" V 3655 2322 50  0000 R CNN
 F 2 "" H 3650 2450 50  0001 C CNN
@@
 $EndComp
 $Comp
-L power:+5V #PWR?
+L power:+5V #PWR03
 U 1 1 5D7A747E
 P 4150 2150
-F 0 "#PWR?" H 4150 2000 50  0001 C CNN
+F 0 "#PWR03" H 4150 2000 50  0001 C CNN
 F 1 "+5V" H 4165 2323 50  0000 C CNN
 F 2 "" H 4150 2150 50  0001 C CNN
@@
 $EndComp
 $Comp
-L Device:R R?
+L Device:R R1
 U 1 1 5D7A74A1
 P 4150 2300
-F 0 "R?" V 3950 2300 50  0000 C CNN
+F 0 "R1" V 3950 2300 50  0000 C CNN
 F 1 "10k" V 4050 2300 50  0000 C CNN
 F 2 "" V 4080 2300 50  0001 C CNN
@@
 $EndComp
 $Comp
-L Device:C C?
+L Device:C C1
 U 1 1 5D7A7D7B
 P 4150 2600
-F 0 "C?" H 4265 2646 50  0000 L CNN
+F 0 "C1" H 4265 2646 50  0000 L CNN
 F 1 "100n" H 4265 2555 50  0000 L CNN
 F 2 "" H 4188 2450 50  0001 C CNN
@@
 Connection ~ 4150 2450
 $Comp
-L power:GND #PWR?
+L power:GND #PWR04
 U 1 1 5D7A7DD1
 P 4150 2750
-F 0 "#PWR?" H 4150 2500 50  0001 C CNN
+F 0 "#PWR04" H 4150 2500 50  0001 C CNN
 F 1 "GND" H 4155 2577 50  0000 C CNN
 F 2 "" H 4150 2750 50  0001 C CNN
@@
 	5200 2450 5200 2900
 $Comp
-L Connector_Generic:Conn_01x10 J?
+L Connector_Generic:Conn_01x10 J2
 U 1 1 5D7A93D5
 P 6900 3300
-F 0 "J?" H 6980 3292 50  0000 L CNN
+F 0 "J2" H 6980 3292 50  0000 L CNN
 F 1 "Conn_01x10" H 6980 3201 50  0000 L CNN
 F 2 "" H 6900 3300 50  0001 C CNN
@@
 $EndComp
 $Comp
-L Connector_Generic:Conn_01x10 J?
+L Connector_Generic:Conn_01x10 J3
 U 1 1 5D7A94CD
 P 6900 4500
-F 0 "J?" H 6980 4492 50  0000 L CNN
+F 0 "J3" H 6980 4492 50  0000 L CNN
 F 1 "Conn_01x10" H 6980 4401 50  0000 L CNN
 F 2 "" H 6900 4500 50  0001 C CNN
@@
 $EndComp
 $Comp
-L Connector_Generic:Conn_01x06 J?
+L Connector_Generic:Conn_01x06 J4
 U 1 1 5D7A9629
 P 6900 5500
-F 0 "J?" H 6980 5492 50  0000 L CNN
+F 0 "J4" H 6980 5492 50  0000 L CNN
 F 1 "Conn_01x06" H 6980 5401 50  0000 L CNN
 F 2 "" H 6900 5500 50  0001 C CNN
